Commit message: - updated fingertip offests to match tech specs of finger tip

File: urdf/left_honda.urdf (robot description, URDF)
Before this commit: robot left_honda, 189 links, 188 joints
Joints:
- joint index_fingertip_attach_joint: origin xyz=0 0 0.0535 rpy=0 0 0 -> xyz=0 0 0.0552 rpy=0 0 0
- joint middle_fingertip_attach_joint: origin xyz=0 0 0.0535 rpy=0 0 0 -> xyz=0 0 0.0552 rpy=0 0 0
- joint ring_fingertip_attach_joint: origin xyz=0 0 0.0535 rpy=0 0 0 -> xyz=0 0 0.0552 rpy=0 0 0
- joint thumb_fingertip_attach_joint: origin xyz=0 0 0.0695 rpy=0 0 0 -> xyz=0 0 0.0712 rpy=0 0 0

File: urdf/left_honda.urdf.xacro (robot description, xacro)
@@ -3,17 +3,17 @@
     <xacro:include filename="$(find allegro_hand_description)/urdf/allegro_hand_description_left.xacro"/>"
     <xacro:include filename="$(find touchlab_description)/urdf/fingertip.xacro"/>"
-    <!-- 0.0155 + 0.038-->
+    <!-- 0.0155 + 0.0397-->
     <xacro:touchlab_fingertip prefix="index_" parent="link_${0*4+3}" size="0.0001">
-        <origin xyz="0 0 0.0535" rpy="0 0 0"/>
+        <origin xyz="0 0 0.0552" rpy="0 0 0"/>
     </xacro:touchlab_fingertip>
     <xacro:touchlab_fingertip prefix="middle_" parent="link_${1*4+3}" size="0.0001">
-        <origin xyz="0 0 0.0535" rpy="0 0 0"/>
+        <origin xyz="0 0 0.0552" rpy="0 0 0"/>
     </xacro:touchlab_fingertip>
     <xacro:touchlab_fingertip prefix="ring_" parent="link_${2*4+3}" size="0.0001">
-        <origin xyz="0 0 0.0535" rpy="0 0 0"/>
+        <origin xyz="0 0 0.0552" rpy="0 0 0"/>
     </xacro:touchlab_fingertip>
-    <!-- 0.0315 + 0.038-->
+    <!-- 0.0315 + 0.0397-->
     <xacro:touchlab_fingertip prefix="thumb_" parent="link_${3*4+3}" size="0.0001">
-        <origin xyz="0 0 0.0695" rpy="0 0 0"/>
+        <origin xyz="0 0 0.0712" rpy="0 0 0"/>
     </xacro:touchlab_fingertip>
 </robot>

File: urdf/right_honda.urdf (robot description, URDF)
Before this commit: robot right_honda, 189 links, 188 joints
Joints:
- joint index_fingertip_attach_joint: origin xyz=0 0 0.0535 rpy=0 0 0 -> xyz=0 0 0.0552 rpy=0 0 0
- joint middle_fingertip_attach_joint: origin xyz=0 0 0.0535 rpy=0 0 0 -> xyz=0 0 0.0552 rpy=0 0 0
- joint ring_fingertip_attach_joint: origin xyz=0 0 0.0535 rpy=0 0 0 -> xyz=0 0 0.0552 rpy=0 0 0
- joint thumb_fingertip_attach_joint: origin xyz=0 0 0.0695 rpy=0 0 0 -> xyz=0 0 0.0712 rpy=0 0 0

File: urdf/right_honda.urdf.xacro (robot description, xacro)
@@ -5,15 +5,15 @@
     <!-- 0.0155 + 0.038-->
     <xacro:touchlab_fingertip prefix="index_" parent="link_${0*4+3}" size="0.0001">
-        <origin xyz="0 0 0.0535" rpy="0 0 0"/>
+        <origin xyz="0 0 0.0552" rpy="0 0 0"/>
     </xacro:touchlab_fingertip>
     <xacro:touchlab_fingertip prefix="middle_" parent="link_${1*4+3}" size="0.0001">
-        <origin xyz="0 0 0.0535" rpy="0 0 0"/>
+        <origin xyz="0 0 0.0552" rpy="0 0 0"/>
     </xacro:touchlab_fingertip>
     <xacro:touchlab_fingertip prefix="ring_" parent="link_${2*4+3}" size="0.0001">
-        <origin xyz="0 0 0.0535" rpy="0 0 0"/>
+        <origin xyz="0 0 0.0552" rpy="0 0 0"/>
     </xacro:touchlab_fingertip>
     <!-- 0.0315 + 0.038-->
     <xacro:touchlab_fingertip prefix="thumb_" parent="link_${3*4+3}" size="0.0001">
-        <origin xyz="0 0 0.0695" rpy="0 0 0"/>
+        <origin xyz="0 0 0.0712" rpy="0 0 0"/>
     </xacro:touchlab_fingertip>
 </robot>
