Commit message: Fix prefixes

File: urdf/allegro_fingertip.xacro (robot description, xacro)
@@ -33,5 +33,5 @@
     </xacro:macro>
     <xacro:macro name="allegro_finger_tip" params="prefix finger_num">
-        <link name="link_${finger_num*4+3}_tip">
+        <link name="${prefix}link_${finger_num*4+3}_tip">
             <visual>
                 <geometry>
@@ -55,7 +55,7 @@
             </inertial>
         </link>
-        <joint name="joint_${finger_num*4+3}_tip" type="fixed">
-            <parent link="link_${finger_num*4+3}"/>
-            <child link="link_${finger_num*4+3}_tip"/>
+        <joint name="${prefix}joint_${finger_num*4+3}_tip" type="fixed">
+            <parent link="${prefix}link_${finger_num*4+3}"/>
+            <child link="${prefix}link_${finger_num*4+3}_tip"/>
             <origin rpy="0 0 0" xyz="0 0 ${link3_z-fingerTip_r}"/>
         </joint>
