Commit message: restructure hand description

File: urdf/allegro_common.xacro (robot description, xacro)
@@ -48,10 +48,10 @@
                  params="prefix finger_num offset_origin_x offset_origin_y offset_origin_z finger_angle_r">
         <!-- [LINK 0, 4, 8] -->
-        <link name="{prefix}link_${finger_num*4+0}">
+        <link name="${prefix}link_${finger_num*4+0}">
             <visual>
                 <geometry>
                     <mesh filename="package://allegro_hand_description/meshes/link_0.0.STL"/>
                 </geometry>
-                <material name="black"/>
+                <material name=""/>
             </visual>
             <collision>
@@ -69,11 +69,11 @@
             </inertial>
         </link>
-        <joint name="{prefix}joint_${finger_num*4+0}" type="revolute">
+        <joint name="${prefix}joint_${finger_num*4+0}" type="revolute">
             <axis xyz="0 0 1"/>
             <limit effort="15" velocity="7"
                    lower="${limit_0_low+joint_safety_margin}"
                    upper="${limit_0_up-joint_safety_margin}"/>
-            <parent link="{prefix}palm_link"/>
-            <child link="{prefix}link_${finger_num*4+0}"/>
+            <parent link="${prefix}palm_link"/>
+            <child link="${prefix}link_${finger_num*4+0}"/>
             <origin rpy="${finger_angle_r} 0 0"
                     xyz="${offset_origin_x} ${offset_origin_y} ${offset_origin_z}"/>
@@ -81,10 +81,10 @@
         </joint>
         <!-- [LINK 1, 5, 9] -->
-        <link name="{prefix}link_${finger_num*4+1}">
+        <link name="${prefix}link_${finger_num*4+1}">
             <visual>
                 <geometry>
                     <mesh filename="package://allegro_hand_description/meshes/link_1.0.STL"/>
                 </geometry>
-                <material name="black"/>
+                <material name=""/>
             </visual>
             <collision>
@@ -102,21 +102,21 @@
             </inertial>
         </link>
-        <joint name="{prefix}joint_${finger_num*4+1}" type="revolute">
+        <joint name="${prefix}joint_${finger_num*4+1}" type="revolute">
             <limit effort="15" velocity="7"
                    lower="${limit_1_low+joint_safety_margin}"
                    upper="${limit_1_up-joint_safety_margin}"/>
             <axis xyz="0 1 0"/>
-            <parent link="{prefix}link_${finger_num*4+0}"/>
-            <child link="{prefix}link_${finger_num*4+1}"/>
+            <parent link="${prefix}link_${finger_num*4+0}"/>
+            <child link="${prefix}link_${finger_num*4+1}"/>
             <origin xyz="0 0 ${link0_z}"/>
             <dynamics damping="3" friction="5"/>
         </joint>
         <!-- [LINK 2, 6, 10]-->
-        <link name="{prefix}link_${finger_num*4+2}">
+        <link name="${prefix}link_${finger_num*4+2}">
             <visual>
                 <geometry>
                     <mesh filename="package://allegro_hand_description/meshes/link_2.0.STL"/>
                 </geometry>
-                <material name="black"/>
+                <material name=""/>
             </visual>
             <collision>
@@ -134,21 +134,21 @@
             </inertial>
         </link>
-        <joint name="{prefix}joint_${finger_num*4+2}" type="revolute">
+        <joint name="${prefix}joint_${finger_num*4+2}" type="revolute">
             <axis xyz="0 1 0"/>
             <limit effort="15" velocity="7"
                    lower="${limit_2_low+joint_safety_margin}"
                    upper="${limit_2_up-joint_safety_margin}"/>
-            <parent link="{prefix}link_${finger_num*4+1}"/>
-            <child link="{prefix}link_${finger_num*4+2}"/>
+            <parent link="${prefix}link_${finger_num*4+1}"/>
+            <child link="${prefix}link_${finger_num*4+2}"/>
             <origin xyz="0 0 ${link1_z}"/>
             <dynamics damping="8" friction="10"/>
         </joint>
         <!-- [LINK 3, 7, 11] -->
-        <link name="{prefix}link_${finger_num*4+3}">
+        <link name="${prefix}link_${finger_num*4+3}">
             <visual>
                 <geometry>
                     <mesh filename="package://allegro_hand_description/meshes/link_3.0.STL"/>
                 </geometry>
-                <material name="black"/>
+                <material name=""/>
             </visual>
             <collision>
@@ -166,11 +166,11 @@
             </inertial>
         </link>
-        <joint name="{prefix}joint_${finger_num*4+3}" type="revolute">
+        <joint name="${prefix}joint_${finger_num*4+3}" type="revolute">
             <axis xyz="0 1 0"/>
             <limit effort="15" velocity="7"
                    lower="${limit_3_low+joint_safety_margin}"
                    upper="${limit_3_up-joint_safety_margin}"/>
-            <parent link="{prefix}link_${finger_num*4+2}"/>
-            <child link="{prefix}link_${finger_num*4+3}"/>
+            <parent link="${prefix}link_${finger_num*4+2}"/>
+            <child link="${prefix}link_${finger_num*4+3}"/>
             <origin xyz="0 0 ${link2_z}"/>
             <dynamics damping="10" friction="12"/>

File: urdf/allegro_fingertip.xacro (robot description, xacro)
@@ -2,5 +2,5 @@
 <robot xmlns:xacro="http://wiki.ros.org/xacro">
     <xacro:include filename="allegro_common.xacro" />
-    <xacro:macro name="allegro_hand_fingertip" params="prefix finger_num origin*">
+    <xacro:macro name="allegro_thumb_tip" params="prefix finger_num">
         <link name="${prefix}link_${finger_num*4+3}_tip">
             <visual>
@@ -32,3 +32,32 @@
         </joint>
     </xacro:macro>
+    <xacro:macro name="allegro_finger_tip" params="prefix finger_num">
+        <link name="link_${finger_num*4+3}_tip">
+            <visual>
+                <geometry>
+                    <mesh filename="package://allegro_hand_description/meshes/link_3.0_tip.STL"/>
+                </geometry>
+                <material name="white">
+                    <color rgba=".9 .9 .9 1"/>
+                </material>
+            </visual>
+            <collision>
+                <geometry>
+                    <sphere radius="${fingerTip_r}"/>
+                </geometry>
+            </collision>
+            <inertial>
+              <mass value="0.0168" />
+              <origin xyz="0 0 0" rpy="0 0 0"/>
+              <inertia ixx="9.68e-07" ixy="0" ixz="0"
+                       iyy="9.68e-07" iyz="0"
+                       izz="9.68e-07" />
+            </inertial>
+        </link>
+        <joint name="joint_${finger_num*4+3}_tip" type="fixed">
+            <parent link="link_${finger_num*4+3}"/>
+            <child link="link_${finger_num*4+3}_tip"/>
+            <origin rpy="0 0 0" xyz="0 0 ${link3_z-fingerTip_r}"/>
+        </joint>
+    </xacro:macro>
 </robot>

File: urdf/allegro_hand_description_left.xacro (robot description, xacro)
@@ -174,5 +174,5 @@
     <!-- RIGHT HAND due to which finger is number 0 -->
     <!-- for LEFT HAND switch the sign of the **offset_origin_y** and **finger_angle_r** parameters-->
-    <xacro:macro name="allegro_hand_left" params="prefix">
+    <xacro:macro name="allegro_hand_left" params="prefix parent *origin">
         <xacro:finger
             prefix="${prefix}"
@@ -210,7 +210,11 @@
             finger_angle_y="${90*DEG2RAD}"
             />
-        <xacro:palm_left
-            prefix="${prefix}"
-            />
+        <xacro:palm_left prefix="${prefix}"/>
+        <joint name="${prefix}palm_attach_joint" type="fixed">
+            <parent link="${parent}"/>
+            <child link="${prefix}palm_link"/>
+            <xacro:insert_block name="origin"/>
+            <axis xyz="0 0 1"/>
+        </joint>
     </xacro:macro>
 </robot>

File: urdf/allegro_hand_description_right.xacro (robot description, xacro)
@@ -174,5 +174,5 @@
     <!-- RIGHT HAND due to which finger is number 0 -->
     <!-- for LEFT HAND switch the sign of the **offset_origin_y** and **finger_angle_r** parameters-->
-    <xacro:macro name="allegro_hand_right" params="prefix">
+    <xacro:macro name="allegro_hand_right" params="prefix parent *origin">
         <xacro:finger
             prefix="${prefix}"
@@ -210,7 +210,11 @@
             finger_angle_y="-${90*DEG2RAD}"
             />
-        <xacro:palm_right
-            prefix="${prefix}"
-            />
+        <xacro:palm_right prefix="${prefix}"/>
+        <joint name="${prefix}palm_attach_joint" type="fixed">
+            <parent link="${parent}"/>
+            <child link="${prefix}palm_link"/>
+            <xacro:insert_block name="origin"/>
+            <axis xyz="0 0 1"/>
+        </joint>
     </xacro:macro>
 </robot>

Commit message: Added torque/velocity limits, adjusted inertias

File: urdf/allegro_common.xacro (robot description, xacro)
@@ -1,4 +1,6 @@
 <?xml version="1.0"?>
 <robot xmlns:xacro="http://www.ros.org/wiki/xacro" name="allegro_hand_left">
+    <xacro:arg name="torque_limit" default="1.0" />
+    <xacro:arg name="velocity_limit" default="5.0" />
     <xacro:property name="DEG2RAD" value="0.01745329251"/>
     <!-- ======================== BASE PARAMS ========================= -->
@@ -44,4 +46,6 @@
     <xacro:property name="limit_3_t_up" value="1.819"/>
     <xacro:property name="limit_3_t_low" value="-0.262"/>
+    <xacro:property name="torque_limit" value="$(arg torque_limit)"/>
+    <xacro:property name="velocity_limit" value="$(arg velocity_limit)"/>
     <!-- THREE FINGER MACRO -->
     <xacro:macro name="finger"
@@ -64,12 +68,12 @@
               <mass value="0.0119" />
               <origin xyz="0 0 0" rpy="0 0 0"/>
-              <inertia ixx="1.01666658333e-06" ixy="0.0" ixz="0.0"
-                       iyy="6.47677333333e-07" iyz="0.0"
-                       izz="1.01666658333e-06" />
+              <inertia ixx="1.01666658333e-4" ixy="0.0" ixz="0.0"
+                       iyy="1.47677333333e-4" iyz="0.0"
+                       izz="1.01666658333e-4" />
             </inertial>
         </link>
         <joint name="${prefix}joint_${finger_num*4+0}" type="revolute">
             <axis xyz="0 0 1"/>
-            <limit effort="15" velocity="7"
+            <limit effort="${torque_limit}" velocity="${velocity_limit}"
                    lower="${limit_0_low+joint_safety_margin}"
                    upper="${limit_0_up-joint_safety_margin}"/>
@@ -97,11 +101,11 @@
               <mass value="0.065" />
               <origin xyz="0 0 0" rpy="0 0 0"/>
-              <inertia ixx="7.95654166667e-05" ixy="1.7199e-05" ixz="8.75875e-06"
-                       iyy="2.47088833333e-05" iyz="2.413125e-05"
-                       izz="7.95654166667e-05" />
+              <inertia ixx="7.95654166667e-4" ixy="0" ixz="0"
+                       iyy="2.47088833333e-4" iyz="0"
+                       izz="7.95654166667e-4" />
             </inertial>
         </link>
         <joint name="${prefix}joint_${finger_num*4+1}" type="revolute">
-            <limit effort="15" velocity="7"
+            <limit effort="${torque_limit}" velocity="${velocity_limit}"
                    lower="${limit_1_low+joint_safety_margin}"
                    upper="${limit_1_up-joint_safety_margin}"/>
@@ -129,12 +133,12 @@
               <mass value="0.0355" />
               <origin xyz="0 0 0" rpy="0 0 0"/>
-              <inertia ixx="2.63979183333e-05" ixy="6.67968e-06" ixz="4.783625e-06"
-                       iyy="1.34948516667e-05" iyz="9.372e-06"
-                       izz="2.63979183333e-05" />
+              <inertia ixx="2.63979183333e-4" ixy="0" ixz="0"
+                       iyy="1.34948516667e-4" iyz="0"
+                       izz="2.63979183333e-4" />
             </inertial>
         </link>
         <joint name="${prefix}joint_${finger_num*4+2}" type="revolute">
             <axis xyz="0 1 0"/>
-            <limit effort="15" velocity="7"
+            <limit effort="${torque_limit}" velocity="${velocity_limit}"
                    lower="${limit_2_low+joint_safety_margin}"
                    upper="${limit_2_up-joint_safety_margin}"/>
@@ -161,12 +165,12 @@
               <mass value="0.0096" />
               <origin xyz="0 0 0" rpy="0 0 0"/>
-              <inertia ixx="4.701248e-06" ixy="1.255968e-06" ixz="1.2936e-06"
-                       iyy="3.649312e-06" iyz="1.7622e-06"
-                       izz="4.701248e-06" />
+              <inertia ixx="4.701248e-4" ixy="0" ixz="0"
+                       iyy="3.649312e-4" iyz="0"
+                       izz="4.701248e-4" />
             </inertial>
         </link>
         <joint name="${prefix}joint_${finger_num*4+3}" type="revolute">
             <axis xyz="0 1 0"/>
-            <limit effort="15" velocity="7"
+            <limit effort="${torque_limit}" velocity="${velocity_limit}"
                    lower="${limit_3_low+joint_safety_margin}"
                    upper="${limit_3_up-joint_safety_margin}"/>

File: urdf/allegro_fingertip.xacro (robot description, xacro)
@@ -21,7 +21,7 @@
               <mass value="0.0168" />
               <origin xyz="0 0 0" rpy="0 0 0"/>
-              <inertia ixx="9.68e-07" ixy="0" ixz="0"
-                       iyy="9.68e-07" iyz="0"
-                       izz="9.68e-07" />
+              <inertia ixx="9.68e-4" ixy="0" ixz="0"
+                       iyy="9.68e-4" iyz="0"
+                       izz="9.68e-4" />
             </inertial>
         </link>
@@ -50,7 +50,7 @@
               <mass value="0.0168" />
               <origin xyz="0 0 0" rpy="0 0 0"/>
-              <inertia ixx="9.68e-07" ixy="0" ixz="0"
-                       iyy="9.68e-07" iyz="0"
-                       izz="9.68e-07" />
+              <inertia ixx="9.68e-4" ixy="0" ixz="0"
+                       iyy="9.68e-4" iyz="0"
+                       izz="9.68e-4" />
             </inertial>
         </link>

File: urdf/allegro_hand_description_left.xacro (robot description, xacro)
@@ -25,12 +25,12 @@
               <mass value="0.0176" />
               <origin xyz="0 0 0" rpy="0 0 0"/>
-              <inertia ixx="1.89273333333e-5" ixy="7.16716e-06" ixz="5.35568e-06"
-                       iyy="1.43008213333e-05" iyz="6.8068e-06"
-                       izz="1.89273333333e-05" />
+              <inertia ixx="1.89273333333e-4" ixy="0" ixz="0"
+                       iyy="1.43008213333e-4" iyz="0"
+                       izz="1.89273333333e-4" />
             </inertial>
         </link>
         <joint name="${prefix}joint_${finger_num*4+0}" type="revolute">
             <axis xyz="+1 0 0"/>
-            <limit effort="15" velocity="7"
+            <limit effort="${torque_limit}" velocity="${velocity_limit}"
                    lower="${limit_0_t_low-joint_safety_margin}"
                    upper="${limit_0_t_up-joint_safety_margin}"/>
@@ -60,12 +60,12 @@
               <mass value="0.0119" />
               <origin xyz="0 0 0" rpy="0 0 0"/>
-              <inertia ixx="4.24250866667e-06" ixy="1.032087e-06" ixz="1.603525e-06"
-                       iyy="4.52362633333e-06" iyz="1.44808125e-06"
-                       izz="4.24250866667e-06" />
+              <inertia ixx="4.24250866667e-4" ixy="0" ixz="0"
+                       iyy="4.52362633333e-4" iyz="0"
+                       izz="4.24250866667e-4" />
             </inertial>
         </link>
         <joint name="${prefix}joint_${finger_num*4+1}" type="revolute">
             <axis xyz="0 0 -1"/>
-            <limit effort="15" velocity="7"
+            <limit effort="${torque_limit}" velocity="${velocity_limit}"
                    lower="${limit_1_t_low+joint_safety_margin}"
                    upper="${limit_1_t_up-joint_safety_margin}"/>
@@ -93,11 +93,12 @@
               <mass value="0.038" />
               <origin xyz="0 0 0" rpy="0 0 0"/>
-              <inertia ixx="4.30439933333e-05" ixy="9.57068e-06" ixz="5.1205e-06" iyy="1.44451933333e-05"
-                       iyz="1.342825e-05" izz="4.30439933333e-05" />
+              <inertia ixx="4.30439933333e-4" ixy="0" ixz="0"
+                       iyy="1.44451933333e-4" iyz="0"
+                       izz="4.30439933333e-4" />
             </inertial>
         </link>
         <joint name="${prefix}joint_${finger_num*4+2}" type="revolute">
             <axis xyz="0 1 0"/>
-            <limit effort="15" velocity="7"
+            <limit effort="${torque_limit}" velocity="${velocity_limit}"
                    lower="${limit_2_t_low+joint_safety_margin}"
                    upper="${limit_2_t_up-joint_safety_margin}"/>
@@ -125,12 +126,12 @@
               <mass value="0.0388" />
               <origin xyz="0 0 0" rpy="0 0 0"/>
-              <inertia ixx="3.29223173333e-05" ixy="8.042076e-06" ixz="5.2283e-06"
-                       iyy="1.47493026667e-5" iyz="1.1283525e-5"
-                       izz="3.29223173333e-05" />
+              <inertia ixx="3.29223173333e-4" ixy="0" ixz="0"
+                       iyy="1.47493026667e-4" iyz="0"
+                       izz="3.29223173333e-4" />
             </inertial>
         </link>
         <joint name="${prefix}joint_${finger_num*4+3}" type="revolute">
             <axis xyz="0 1 0"/>
-            <limit effort="15" velocity="7"
+            <limit effort="${torque_limit}" velocity="${velocity_limit}"
                    lower="${limit_3_t_low+joint_safety_margin}"
                    upper="${limit_3_t_up-joint_safety_margin}"/>

File: urdf/allegro_hand_description_right.xacro (robot description, xacro)
@@ -25,12 +25,12 @@
               <mass value="0.0176" />
               <origin xyz="0 0 0" rpy="0 0 0"/>
-              <inertia ixx="1.89273333333e-5" ixy="7.16716e-06" ixz="5.35568e-06"
-                       iyy="1.43008213333e-05" iyz="6.8068e-06"
-                       izz="1.89273333333e-05" />
+              <inertia ixx="1.89273333333e-4" ixy="0" ixz="0"
+                       iyy="1.43008213333e-4" iyz="0"
+                       izz="1.89273333333e-4" />
             </inertial>
         </link>
         <joint name="${prefix}joint_${finger_num*4+0}" type="revolute">
             <axis xyz="-1 0 0"/>
-            <limit effort="15" velocity="7"
+            <limit effort="${torque_limit}" velocity="${velocity_limit}"
                    lower="${limit_0_t_low-joint_safety_margin}"
                    upper="${limit_0_t_up-joint_safety_margin}"/>
@@ -60,12 +60,12 @@
               <mass value="0.0119" />
               <origin xyz="0 0 0" rpy="0 0 0"/>
-              <inertia ixx="4.24250866667e-06" ixy="1.032087e-06" ixz="1.603525e-06"
-                       iyy="4.52362633333e-06" iyz="1.44808125e-06"
-                       izz="4.24250866667e-06" />
+              <inertia ixx="4.24250866667e-4" ixy="0" ixz="0"
+                       iyy="4.52362633333e-4" iyz="0"
+                       izz="4.24250866667e-4" />
             </inertial>
         </link>
         <joint name="${prefix}joint_${finger_num*4+1}" type="revolute">
             <axis xyz="0 0 1"/>
-            <limit effort="15" velocity="7"
+            <limit effort="${torque_limit}" velocity="${velocity_limit}"
                    lower="${limit_1_t_low+joint_safety_margin}"
                    upper="${limit_1_t_up-joint_safety_margin}"/>
@@ -93,11 +93,12 @@
               <mass value="0.038" />
               <origin xyz="0 0 0" rpy="0 0 0"/>
-              <inertia ixx="4.30439933333e-05" ixy="9.57068e-06" ixz="5.1205e-06" iyy="1.44451933333e-05"
-                       iyz="1.342825e-05" izz="4.30439933333e-05" />
+              <inertia ixx="4.30439933333e-4" ixy="0" ixz="0"
+                       iyy="1.44451933333e-4" iyz="0"
+                       izz="4.30439933333e-4" />
             </inertial>
         </link>
         <joint name="${prefix}joint_${finger_num*4+2}" type="revolute">
             <axis xyz="0 1 0"/>
-            <limit effort="15" velocity="7"
+            <limit effort="${torque_limit}" velocity="${velocity_limit}"
                    lower="${limit_2_t_low+joint_safety_margin}"
                    upper="${limit_2_t_up-joint_safety_margin}"/>
@@ -125,12 +126,12 @@
               <mass value="0.0388" />
               <origin xyz="0 0 0" rpy="0 0 0"/>
-              <inertia ixx="3.29223173333e-05" ixy="8.042076e-06" ixz="5.2283e-06"
-                       iyy="1.47493026667e-5" iyz="1.1283525e-5"
-                       izz="3.29223173333e-05" />
+              <inertia ixx="3.29223173333e-4" ixy="0" ixz="0"
+                       iyy="1.47493026667e-4" iyz="0"
+                       izz="3.29223173333e-4" />
             </inertial>
         </link>
         <joint name="${prefix}joint_${finger_num*4+3}" type="revolute">
             <axis xyz="0 1 0"/>
-            <limit effort="15" velocity="7"
+            <limit effort="${torque_limit}" velocity="${velocity_limit}"
                    lower="${limit_3_t_low+joint_safety_margin}"
                    upper="${limit_3_t_up-joint_safety_margin}"/>
@@ -161,10 +162,10 @@
             </collision>
             <inertial>
-            <origin xyz="0 0 ${palm_link_z/2}" rpy="0 0 0"/>
-            <mass value="0.4154"/>
-            <inertia
-                ixx="1e-4" ixy="0.0" ixz="0.0"
-                iyy="1e-4" iyz="0.0"
-                izz="1e-4"/>
+                <origin xyz="0 0 ${palm_link_z/2}" rpy="0 0 0"/>
+                <mass value="0.4154"/>
+                <inertia
+                    ixx="1e-4" ixy="0.0" ixz="0.0"
+                    iyy="1e-4" iyz="0.0"
+                    izz="1e-4"/>
             </inertial>
         </link>
