Commit message: renamed all the stl and the codes

File: urdf/allegro_common.xacro (robot description, xacro)
@@ -55,5 +55,5 @@
             <visual>
                 <geometry>
-                    <mesh filename="package://allegro_hand_description/meshes/link_0.0.STL"/>
+                    <mesh filename="package://allegro_hand_description/meshes/link_0_0.STL"/>
                 </geometry>
                 <material name=""/>
@@ -88,5 +88,5 @@
             <visual>
                 <geometry>
-                    <mesh filename="package://allegro_hand_description/meshes/link_1.0.STL"/>
+                    <mesh filename="package://allegro_hand_description/meshes/link_1_0.STL"/>
                 </geometry>
                 <material name=""/>
@@ -120,5 +120,5 @@
             <visual>
                 <geometry>
-                    <mesh filename="package://allegro_hand_description/meshes/link_2.0.STL"/>
+                    <mesh filename="package://allegro_hand_description/meshes/link_2_0.STL"/>
                 </geometry>
                 <material name=""/>
@@ -152,5 +152,5 @@
             <visual>
                 <geometry>
-                    <mesh filename="package://allegro_hand_description/meshes/link_3.0.STL"/>
+                    <mesh filename="package://allegro_hand_description/meshes/link_3_0.STL"/>
                 </geometry>
                 <material name=""/>

File: urdf/allegro_fingertip.xacro (robot description, xacro)
@@ -6,5 +6,5 @@
             <visual>
                 <geometry>
-                    <mesh filename="package://allegro_hand_description/meshes/link_15.0_tip.STL"/>
+                    <mesh filename="package://allegro_hand_description/meshes/link_15_0_tip.STL"/>
                 </geometry>
                 <material name="white">
@@ -36,5 +36,5 @@
             <visual>
                 <geometry>
-                    <mesh filename="package://allegro_hand_description/meshes/link_3.0_tip.STL"/>
+                    <mesh filename="package://allegro_hand_description/meshes/link_3_0_tip.STL"/>
                 </geometry>
                 <material name="white">

File: urdf/allegro_hand_description_left.xacro (robot description, xacro)
@@ -9,5 +9,5 @@
             <visual>
                 <geometry>
-                    <mesh filename="package://allegro_hand_description/meshes/link_12.0_left.STL"/>
+                    <mesh filename="package://allegro_hand_description/meshes/link_12_0_left.STL"/>
                 </geometry>
                 <material name="black">
@@ -45,5 +45,5 @@
             <visual>
                 <geometry>
-                    <mesh filename="package://allegro_hand_description/meshes/link_13.0.STL"/>
+                    <mesh filename="package://allegro_hand_description/meshes/link_13_0.STL"/>
                 </geometry>
                 <material name="black">
@@ -79,5 +79,5 @@
             <visual>
                 <geometry>
-                    <mesh filename="package://allegro_hand_description/meshes/link_14.0.STL"/>
+                    <mesh filename="package://allegro_hand_description/meshes/link_14_0.STL"/>
                 </geometry>
                 <material name="black">
@@ -112,5 +112,5 @@
             <visual>
                 <geometry>
-                    <mesh filename="package://allegro_hand_description/meshes/link_15.0.STL"/>
+                    <mesh filename="package://allegro_hand_description/meshes/link_15_0.STL"/>
                 </geometry>
                 <material name="black">

File: urdf/allegro_hand_description_right.xacro (robot description, xacro)
@@ -9,5 +9,5 @@
             <visual>
                 <geometry>
-                    <mesh filename="package://allegro_hand_description/meshes/link_12.0_right.STL"/>
+                    <mesh filename="package://allegro_hand_description/meshes/link_12_0_right.STL"/>
                 </geometry>
                 <material name="black">
@@ -45,5 +45,5 @@
             <visual>
                 <geometry>
-                    <mesh filename="package://allegro_hand_description/meshes/link_13.0.STL"/>
+                    <mesh filename="package://allegro_hand_description/meshes/link_13_0.STL"/>
                 </geometry>
                 <material name="black">
@@ -79,5 +79,5 @@
             <visual>
                 <geometry>
-                    <mesh filename="package://allegro_hand_description/meshes/link_14.0.STL"/>
+                    <mesh filename="package://allegro_hand_description/meshes/link_14_0.STL"/>
                 </geometry>
                 <material name="black">
@@ -112,5 +112,5 @@
             <visual>
                 <geometry>
-                    <mesh filename="package://allegro_hand_description/meshes/link_15.0.STL"/>
+                    <mesh filename="package://allegro_hand_description/meshes/link_15_0.STL"/>
                 </geometry>
                 <material name="black">

Commit message: renamed all the stl and the codes

File: urdf/allegro_common.xacro (robot description, xacro)
@@ -51,5 +51,5 @@
             <visual>
                 <geometry>
-                    <mesh filename="package://allegro_hand_description/meshes/link_0.0.STL"/>
+                    <mesh filename="package://allegro_hand_description/meshes/link_0_0.STL"/>
                 </geometry>
                 <material name=""/>
@@ -84,5 +84,5 @@
             <visual>
                 <geometry>
-                    <mesh filename="package://allegro_hand_description/meshes/link_1.0.STL"/>
+                    <mesh filename="package://allegro_hand_description/meshes/link_1_0.STL"/>
                 </geometry>
                 <material name=""/>
@@ -116,5 +116,5 @@
             <visual>
                 <geometry>
-                    <mesh filename="package://allegro_hand_description/meshes/link_2.0.STL"/>
+                    <mesh filename="package://allegro_hand_description/meshes/link_2_0.STL"/>
                 </geometry>
                 <material name=""/>
@@ -148,5 +148,5 @@
             <visual>
                 <geometry>
-                    <mesh filename="package://allegro_hand_description/meshes/link_3.0.STL"/>
+                    <mesh filename="package://allegro_hand_description/meshes/link_3_0.STL"/>
                 </geometry>
                 <material name=""/>

File: urdf/allegro_fingertip.xacro (robot description, xacro)
@@ -6,5 +6,5 @@
             <visual>
                 <geometry>
-                    <mesh filename="package://allegro_hand_description/meshes/link_15.0_tip.STL"/>
+                    <mesh filename="package://allegro_hand_description/meshes/link_15_0_tip.STL"/>
                 </geometry>
                 <material name="white">
@@ -36,5 +36,5 @@
             <visual>
                 <geometry>
-                    <mesh filename="package://allegro_hand_description/meshes/link_3.0_tip.STL"/>
+                    <mesh filename="package://allegro_hand_description/meshes/link_3_0_tip.STL"/>
                 </geometry>
                 <material name="white">

File: urdf/allegro_hand_description_left.xacro (robot description, xacro)
@@ -9,5 +9,5 @@
             <visual>
                 <geometry>
-                    <mesh filename="package://allegro_hand_description/meshes/link_12.0_left.STL"/>
+                    <mesh filename="package://allegro_hand_description/meshes/link_12_0_left.STL"/>
                 </geometry>
                 <material name="black">
@@ -45,5 +45,5 @@
             <visual>
                 <geometry>
-                    <mesh filename="package://allegro_hand_description/meshes/link_13.0.STL"/>
+                    <mesh filename="package://allegro_hand_description/meshes/link_13_0.STL"/>
                 </geometry>
                 <material name="black">
@@ -79,5 +79,5 @@
             <visual>
                 <geometry>
-                    <mesh filename="package://allegro_hand_description/meshes/link_14.0.STL"/>
+                    <mesh filename="package://allegro_hand_description/meshes/link_14_0.STL"/>
                 </geometry>
                 <material name="black">
@@ -111,5 +111,5 @@
             <visual>
                 <geometry>
-                    <mesh filename="package://allegro_hand_description/meshes/link_15.0.STL"/>
+                    <mesh filename="package://allegro_hand_description/meshes/link_15_0.STL"/>
                 </geometry>
                 <material name="black">

File: urdf/allegro_hand_description_right.xacro (robot description, xacro)
@@ -9,5 +9,5 @@
             <visual>
                 <geometry>
-                    <mesh filename="package://allegro_hand_description/meshes/link_12.0_right.STL"/>
+                    <mesh filename="package://allegro_hand_description/meshes/link_12_0_right.STL"/>
                 </geometry>
                 <material name="black">
@@ -45,5 +45,5 @@
             <visual>
                 <geometry>
-                    <mesh filename="package://allegro_hand_description/meshes/link_13.0.STL"/>
+                    <mesh filename="package://allegro_hand_description/meshes/link_13_0.STL"/>
                 </geometry>
                 <material name="black">
@@ -79,5 +79,5 @@
             <visual>
                 <geometry>
-                    <mesh filename="package://allegro_hand_description/meshes/link_14.0.STL"/>
+                    <mesh filename="package://allegro_hand_description/meshes/link_14_0.STL"/>
                 </geometry>
                 <material name="black">
@@ -111,5 +111,5 @@
             <visual>
                 <geometry>
-                    <mesh filename="package://allegro_hand_description/meshes/link_15.0.STL"/>
+                    <mesh filename="package://allegro_hand_description/meshes/link_15_0.STL"/>
                 </geometry>
                 <material name="black">
