Commit message: allegro right hand ros2 control

File: ros2_control/allegro.ros2_control.xacro (robot description, xacro)
@@ -8,5 +8,5 @@
     </joint>
   </xacro:macro>
-  <xacro:macro name="allegro_ros2_control" params="name prefix port hand_id use_mock_hardware:=^|false">
+  <xacro:macro name="allegro_ros2_control" params="name prefix port hand_id use_mock_hardware">
     <ros2_control name="${name}" type="system">
       <xacro:unless value="${use_mock_hardware}">
@@ -23,20 +23,20 @@
         </hardware>
       </xacro:if>
-      <xacro:joint_hw joint_num="0"/>
-      <xacro:joint_hw joint_num="1"/>
-      <xacro:joint_hw joint_num="2"/>
-      <xacro:joint_hw joint_num="3"/>
-      <xacro:joint_hw joint_num="4"/>
-      <xacro:joint_hw joint_num="5"/>
-      <xacro:joint_hw joint_num="6"/>
-      <xacro:joint_hw joint_num="7"/>
-      <xacro:joint_hw joint_num="8"/>
-      <xacro:joint_hw joint_num="9"/>
-      <xacro:joint_hw joint_num="10"/>
-      <xacro:joint_hw joint_num="11"/>
-      <xacro:joint_hw joint_num="12"/>
-      <xacro:joint_hw joint_num="13"/>
-      <xacro:joint_hw joint_num="14"/>
-      <xacro:joint_hw joint_num="15"/>
+      <xacro:joint_hw joint_num="0" prefix="${prefix}"/>
+      <xacro:joint_hw joint_num="1" prefix="${prefix}"/>
+      <xacro:joint_hw joint_num="2" prefix="${prefix}"/>
+      <xacro:joint_hw joint_num="3" prefix="${prefix}"/>
+      <xacro:joint_hw joint_num="4" prefix="${prefix}"/>
+      <xacro:joint_hw joint_num="5" prefix="${prefix}"/>
+      <xacro:joint_hw joint_num="6" prefix="${prefix}"/>
+      <xacro:joint_hw joint_num="7" prefix="${prefix}"/>
+      <xacro:joint_hw joint_num="8" prefix="${prefix}"/>
+      <xacro:joint_hw joint_num="9" prefix="${prefix}"/>
+      <xacro:joint_hw joint_num="10" prefix="${prefix}"/>
+      <xacro:joint_hw joint_num="11" prefix="${prefix}"/>
+      <xacro:joint_hw joint_num="12" prefix="${prefix}"/>
+      <xacro:joint_hw joint_num="13" prefix="${prefix}"/>
+      <xacro:joint_hw joint_num="14" prefix="${prefix}"/>
+      <xacro:joint_hw joint_num="15" prefix="${prefix}"/>
     </ros2_control>
   </xacro:macro>

File: urdf/allegro_hand_right.urdf.xacro (robot description, xacro)
@@ -7,5 +7,5 @@
     <xacro:include filename="allegro_hand_description_right.xacro"/>
     <xacro:include filename="allegro_fingertip.xacro"/>
-    <xacro::include filename="$(find allegro_hand_description)/ros2_control/allegro.ros2_control.xacro"/>
+    <xacro:include filename="$(find allegro_hand_description)/ros2_control/allegro.ros2_control.xacro"/>
     <link name="world"></link>
     <xacro:allegro_hand_right prefix="$(arg prefix)" parent="world">

Commit message: Added filtering params

File: ros2_control/allegro.ros2_control.xacro (robot description, xacro)
@@ -8,5 +8,5 @@
     </joint>
   </xacro:macro>
-  <xacro:macro name="allegro_ros2_control" params="name prefix port hand_id use_mock_hardware">
+  <xacro:macro name="allegro_ros2_control" params="name prefix port hand_id use_mock_hardware position_filtering velocity_filtering">
     <ros2_control name="${name}" type="system">
       <hardware>
@@ -15,4 +15,6 @@
           <param name="port">${port}</param>
           <param name="hand_id">${hand_id}</param>
+          <param name="position_filtering">${position_filtering}</param>
+          <param name="velocity_filtering">${velocity_filtering}</param>
           <param name="joint_0_offset">0.0</param>
           <param name="joint_1_offset">0.0</param>
